Commit message: tool scaled and correctly allocated. TCP should be calculated

File: fanuc_experimental/fanuc_lrmate200id_support/urdf/spray_tool.xacro (robot description, xacro)
@@ -1,29 +1,24 @@
 <?xml version="1.0" encoding="utf-8"?>
 <robot xmlns:xacro="http://ros.org/wiki/xacro">
-  <!-- Here we define the 2 parameters of the macro -->
   <xacro:macro name="spray_tool" params="prefix connected_to">
     <!-- Create a fixed joint with a parameterized name. -->
     <joint name="${prefix}spray_tool_joint" type="fixed">
-      <!-- The parent link must be read from the robot model it is attached to. -->
-      <parent link="${connected_to}"/>
+<!-- Copied from original data    <parent link="${connected_to}"/> -->
+      <parent link="${prefix}flange"/>
       <child link="${prefix}spray_tool"/>
-      <!-- The tool is directly attached to the flange. -->
-      <origin rpy="0 0 0" xyz="0 0 0"/>
+      <origin rpy="${-pi/2} 0 ${pi}" xyz="0 0 0"/>
     </joint>
     <link name="${prefix}spray_tool">
       <visual>
         <geometry>
-          <!-- The path to the visual meshes in the package. -->
-          <mesh filename="file://$(find fanuc_lrmate200id_support)/meshes/lrmate200id/visual/spray_tool.stl"/>
+          <mesh filename="file://$(find fanuc_lrmate200id_support)/meshes/lrmate200id/visual/spray_tool2.stl" scale="0.001 0.001 0.001"/>
         </geometry>
       </visual>
       <collision>
         <geometry>
-          <!-- The path to the collision meshes in the package. -->
-          <mesh filename="file://$(find fanuc_lrmate200id_support)/meshes/lrmate200id/visual/spray_tool.stl"/>
+          <mesh filename="file://$(find fanuc_lrmate200id_support)/meshes/lrmate200id/visual/spray_tool2.stl" scale="0.001 0.001 0.001"/>
         </geometry>
       </collision>
     </link>
-    <!-- TCP frame -->
     <joint name="${prefix}tcp_joint" type="fixed">
       <origin xyz="0 0 0.116" rpy="0 0 0"/>

Commit message: cleaned

File: fanuc_experimental/fanuc_lrmate200id_support/urdf/spray_tool.xacro (robot description, xacro)
@@ -4,5 +4,4 @@
         <!-- Create a fixed joint with a parameterized name. -->
         <joint name="${prefix}spray_tool_joint" type="fixed">
-            <!-- Copied from original data    <parent link="${connected_to}"/> -->
             <parent link="${prefix}tool0"/>
             <child link="${prefix}spray_tool"/>
