Commit message: added visualization of tool

File: fanuc_experimental/fanuc_lrmate200id_support/urdf/lrmate200id.xacro (robot description, xacro)
@@ -4,8 +4,11 @@
   <xacro:fanuc_lrmate200id prefix=""/>
     <!--Import the asus xtion macro -->
-     <xacro:include filename="$(find realsense2_description)/urdf/_d435.urdf.xacro"/>
-  <xacro:sensor_d435 parent="base_link">
-    <origin xyz="0.2 0.2 0.2" rpy="0 0 0"/>
-  </xacro:sensor_d435>
+<!--     <xacro:include filename="$(find realsense2_description)/urdf/_d435.urdf.xacro"/> -->
+<!--  <xacro:sensor_d435 parent="base_link">-->
+<!--    <origin xyz="0.2 0.2 0.2" rpy="0 0 0"/>-->
+<!--  </xacro:sensor_d435>-->
+<!--  <xacro:spray_tool prefix="" connected_to="tool0"/>-->
+ <xacro:include filename="$(find fanuc_lrmate200id_support)/urdf/spray_tool.xacro"/>
+      <xacro:spray_tool prefix="" connected_to="tool0"/>
   <link name="world" />
   <joint name="world_joint" type="fixed">

Commit message: tcp is calculated. orientation problems are met

File: fanuc_experimental/fanuc_lrmate200id_support/urdf/lrmate200id.xacro (robot description, xacro)
@@ -4,11 +4,10 @@
   <xacro:fanuc_lrmate200id prefix=""/>
     <!--Import the asus xtion macro -->
-<!--     <xacro:include filename="$(find realsense2_description)/urdf/_d435.urdf.xacro"/> -->
-<!--  <xacro:sensor_d435 parent="base_link">-->
-<!--    <origin xyz="0.2 0.2 0.2" rpy="0 0 0"/>-->
-<!--  </xacro:sensor_d435>-->
-<!--  <xacro:spray_tool prefix="" connected_to="tool0"/>-->
+     <xacro:include filename="$(find realsense2_description)/urdf/_d435.urdf.xacro"/>
+  <xacro:sensor_d435 parent="base_link">
+    <origin xyz="0.15 0.0 0.2" rpy="0 0 0"/>
+  </xacro:sensor_d435>
  <xacro:include filename="$(find fanuc_lrmate200id_support)/urdf/spray_tool.xacro"/>
-      <xacro:spray_tool prefix="" connected_to="tool0"/>
+      <xacro:spray_tool prefix="" connected_to="flange"/>
   <link name="world" />
   <joint name="world_joint" type="fixed">

File: fanuc_experimental/fanuc_lrmate200id_support/urdf/lrmate200id_macro.xacro (robot description, xacro)
@@ -167,10 +167,10 @@
     </joint>
     <!-- ROS-Industrial 'tool0' frame: all-zeros tool frame -->
-    <link name="${prefix}tool0" />
-    <joint name="${prefix}link_6-tool0" type="fixed">
-      <origin xyz="0 0 0" rpy="${pi} ${-pi/2.0} 0" />
-      <parent link="${prefix}flange" />
-      <child link="${prefix}tool0" />
-    </joint>
+<!--    <link name="${prefix}tool0" />-->
+<!--    <joint name="${prefix}link_6-tool0" type="fixed">-->
+<!--      <origin xyz="0 0 0" rpy="${pi} ${-pi/2.0} 0" />-->
+<!--      <parent link="${prefix}flange" />-->
+<!--      <child link="${prefix}tool0" />-->
+<!--    </joint>-->
   </xacro:macro>
 </robot>

File: fanuc_experimental/fanuc_lrmate200id_support/urdf/spray_tool.xacro (robot description, xacro)
@@ -12,15 +12,15 @@
       <visual>
         <geometry>
-          <mesh filename="file://$(find fanuc_lrmate200id_support)/meshes/lrmate200id/visual/spray_tool2.stl" scale="0.001 0.001 0.001"/>
+          <mesh filename="file://$(find fanuc_lrmate200id_support)/meshes/lrmate200id/visual/spray_tool.stl" scale="0.001 0.001 0.001"/>
         </geometry>
       </visual>
-      <collision>
-        <geometry>
-          <mesh filename="file://$(find fanuc_lrmate200id_support)/meshes/lrmate200id/visual/spray_tool2.stl" scale="0.001 0.001 0.001"/>
-        </geometry>
-      </collision>
+<!--      <collision>-->
+<!--        <geometry>-->
+<!--          <mesh filename="file://$(find fanuc_lrmate200id_support)/meshes/lrmate200id/visual/spray_tool.stl" scale="0.001 0.001 0.001"/>-->
+<!--        </geometry>-->
+<!--      </collision>-->
     </link>
     <joint name="${prefix}tcp_joint" type="fixed">
-      <origin xyz="0 0 0.116" rpy="0 0 0"/>
+      <origin xyz="-0.0758 0 0.2" rpy="0 0 0"/>
       <parent link="${prefix}spray_tool"/>
       <child link="${prefix}tcp"/>

Commit message: kinematics solver switched, robot description files updated

File: fanuc_experimental/fanuc_lrmate200id_support/urdf/lrmate200id.xacro (robot description, xacro)
@@ -1,18 +1,23 @@
 <?xml version="1.0"?>
 <robot name="fanuc_lrmate200id" xmlns:xacro="http://wiki.ros.org/xacro">
-  <xacro:include filename="$(find fanuc_lrmate200id_support)/urdf/lrmate200id_macro.xacro"/>
-  <xacro:fanuc_lrmate200id prefix=""/>
-    <!--Import the asus xtion macro -->
-     <xacro:include filename="$(find realsense2_description)/urdf/_d435.urdf.xacro"/>
-  <xacro:sensor_d435 parent="base_link">
-    <origin xyz="0.15 0.0 0.2" rpy="0 0 0"/>
-  </xacro:sensor_d435>
- <xacro:include filename="$(find fanuc_lrmate200id_support)/urdf/spray_tool.xacro"/>
-      <xacro:spray_tool prefix="" connected_to="flange"/>
-  <link name="world" />
-  <joint name="world_joint" type="fixed">
-    <parent link="world" />
-    <child link = "base_link" />
-    <origin xyz="0.0 0.0 0.0" rpy="0.0 0.0 0.0" />
-  </joint>
+    <xacro:include filename="$(find fanuc_lrmate200id_support)/urdf/lrmate200id_macro.xacro"/>
+    <xacro:fanuc_lrmate200id prefix=""/>
+    <xacro:include filename="$(find realsense2_description)/urdf/_d435.urdf.xacro"/>
+    <xacro:sensor_d435 parent="base_link">
+        <origin xyz="0.15 0.0 0.2" rpy="0 0 0"/>
+    </xacro:sensor_d435>
+    <xacro:include filename="$(find fanuc_lrmate200id_support)/urdf/spray_tool.xacro"/>
+    <xacro:spray_tool prefix="" connected_to=""/>
+    <link name="tcp"/>
+    <joint name="tcp_joint" type="fixed">
+        <origin xyz="-0.0758 0 0.2" rpy="0 0 ${pi}"/>
+        <parent link="spray_tool"/>
+        <child link="tcp"/>
+    </joint>
+    <link name="world"/>
+    <joint name="world_joint" type="fixed">
+        <parent link="world"/>
+        <child link="base_link"/>
+        <origin xyz="0.0 0.0 0.0" rpy="0.0 0.0 0.0"/>
+    </joint>
 </robot>

File: fanuc_experimental/fanuc_lrmate200id_support/urdf/lrmate200id_macro.xacro (robot description, xacro)
@@ -1,176 +1,176 @@
 <?xml version="1.0"?>
 <robot xmlns:xacro="http://wiki.ros.org/xacro">
-  <xacro:include filename="$(find fanuc_resources)/urdf/common_materials.xacro"/>
-  <xacro:macro name="fanuc_lrmate200id" params="prefix">
-    <!-- links: main serial chain -->
-    <link name="${prefix}base_link">
-      <visual>
-        <origin xyz="0 0 0" rpy="0 0 0"/>
-        <geometry>
-          <mesh filename="package://fanuc_lrmate200id_support/meshes/lrmate200id/visual/base_link.stl"/>
-        </geometry>
-        <xacro:material_fanuc_gray28 />
-      </visual>
-      <collision>
-        <origin xyz="0 0 0" rpy="0 0 0"/>
-        <geometry>
-          <mesh filename="package://fanuc_lrmate200id_support/meshes/lrmate200id/collision/base_link.stl"/>
-        </geometry>
-      </collision>
-    </link>
-    <link name="${prefix}link_1">
-      <visual>
-        <origin xyz="0 0 0" rpy="0 0 0"/>
-        <geometry>
-          <mesh filename="package://fanuc_lrmate200id_support/meshes/lrmate200id/visual/link_1.stl"/>
-        </geometry>
-        <xacro:material_fanuc_yellow />
-      </visual>
-      <collision>
-        <origin xyz="0 0 0" rpy="0 0 0"/>
-        <geometry>
-          <mesh filename="package://fanuc_lrmate200id_support/meshes/lrmate200id/collision/link_1.stl"/>
-        </geometry>
-      </collision>
-    </link>
-    <link name="${prefix}link_2">
-      <visual>
-        <origin xyz="0 0 0" rpy="0 0 0"/>
-        <geometry>
-          <mesh filename="package://fanuc_lrmate200id_support/meshes/lrmate200id/visual/link_2.stl"/>
-        </geometry>
-        <xacro:material_fanuc_yellow />
-      </visual>
-      <collision>
-        <origin xyz="0 0 0" rpy="0 0 0"/>
-        <geometry>
-          <mesh filename="package://fanuc_lrmate200id_support/meshes/lrmate200id/collision/link_2.stl"/>
-        </geometry>
-      </collision>
-    </link>
-    <link name="${prefix}link_3">
-      <visual>
-        <origin xyz="0 0 0" rpy="0 0 0"/>
-        <geometry>
-          <mesh filename="package://fanuc_lrmate200id_support/meshes/lrmate200id/visual/link_3.stl"/>
-        </geometry>
-        <xacro:material_fanuc_yellow />
-      </visual>
-      <collision>
-        <origin xyz="0 0 0" rpy="0 0 0"/>
-        <geometry>
-          <mesh filename="package://fanuc_lrmate200id_support/meshes/lrmate200id/collision/link_3.stl"/>
-        </geometry>
-      </collision>
-    </link>
-    <link name="${prefix}link_4">
-      <visual>
-        <origin xyz="0 0 0" rpy="0 0 0"/>
-        <geometry>
-          <mesh filename="package://fanuc_lrmate200id_support/meshes/lrmate200id/visual/link_4.stl"/>
-        </geometry>
-        <xacro:material_fanuc_yellow />
-      </visual>
-      <collision>
-        <origin xyz="0 0 0" rpy="0 0 0"/>
-        <geometry>
-          <mesh filename="package://fanuc_lrmate200id_support/meshes/lrmate200id/collision/link_4.stl"/>
-        </geometry>
-      </collision>
-    </link>
-    <link name="${prefix}link_5">
-      <visual>
-        <origin xyz="0 0 0" rpy="0 0 0"/>
-        <geometry>
-          <mesh filename="package://fanuc_lrmate200id_support/meshes/lrmate200id/visual/link_5.stl"/>
-        </geometry>
-        <xacro:material_fanuc_yellow />
-      </visual>
-      <collision>
-        <origin xyz="0 0 0" rpy="0 0 0"/>
-        <geometry>
-          <mesh filename="package://fanuc_lrmate200id_support/meshes/lrmate200id/collision/link_5.stl"/>
-        </geometry>
-      </collision>
-    </link>
-    <link name="${prefix}link_6">
-      <visual>
-        <origin xyz="0 0 0" rpy="0 0 0"/>
-        <geometry>
-          <mesh filename="package://fanuc_lrmate200id_support/meshes/lrmate200id/visual/link_6.stl"/>
-        </geometry>
-        <xacro:material_fanuc_black />
-      </visual>
-      <collision>
-        <origin xyz="0 0 0" rpy="0 0 0"/>
-        <geometry>
-          <mesh filename="package://fanuc_lrmate200id_support/meshes/lrmate200id/collision/link_6.stl"/>
-        </geometry>
-      </collision>
-    </link>
-    <!-- joints: main serial chain -->
-    <joint name="${prefix}joint_1" type="revolute">
-      <origin xyz="0 0 0.330" rpy="0 0 0" />
-      <parent link="${prefix}base_link" />
-      <child link="${prefix}link_1" />
-      <axis xyz="0 0 1" />
-      <limit effort="0" lower="-2.965" upper="2.965" velocity="7.85" />
-    </joint>
-    <joint name="${prefix}joint_2" type="revolute">
-      <origin xyz="0.050 0 0" rpy="0 0 0"/>
-      <parent link="${prefix}link_1" />
-      <child link="${prefix}link_2" />
-      <axis xyz="0 1 0" />
-      <limit effort="0" lower="-1.745329" upper="2.530727" velocity="6.63" />
-    </joint>
-    <joint name="${prefix}joint_3" type="revolute">
-      <origin xyz="0 0 0.330" rpy="0 0 0"/>
-      <parent link="${prefix}link_2" />
-      <child link="${prefix}link_3" />
-      <axis xyz="0 -1 0" />
-      <limit effort="0" lower="-2.450966" upper="4.886922" velocity="9.08" />
-    </joint>
-    <joint name="${prefix}joint_4" type="revolute">
-      <origin xyz="0 0 0.035" rpy="0 0 0"/>
-      <parent link="${prefix}link_3"/>
-      <child link="${prefix}link_4"/>
-      <axis xyz="-1 0 0"/>
-      <limit effort="0" lower="-3.315" upper="3.315" velocity="9.60" />
-    </joint>
-    <joint name="${prefix}joint_5" type="revolute">
-      <origin xyz="0.335 0 0" rpy="0 0 0"/>
-      <parent link="${prefix}link_4"/>
-      <child link="${prefix}link_5"/>
-      <axis xyz="0 -1 0"/>
-      <limit effort="0" lower="-2.18" upper="2.18" velocity="9.51" />
-    </joint>
-    <joint name="${prefix}joint_6" type="revolute">
-      <origin xyz="0.080 0 0" rpy="0 0 0"/>
-      <parent link="${prefix}link_5"/>
-      <child link="${prefix}link_6"/>
-      <axis xyz="-1 0 0"/>
-      <limit effort="0" lower="-6.285" upper="6.285" velocity="17.45" />
-    </joint>
-    <!-- ROS-Industrial 'base' frame: base_link to Fanuc World Coordinates transform -->
-    <link name="${prefix}base" />
-    <joint name="${prefix}base_link-base" type="fixed">
-      <origin xyz="0 0 0.330" rpy="0 0 0"/>
-      <parent link="${prefix}base_link"/>
-      <child link="${prefix}base"/>
-    </joint>
-    <!-- ROS-Industrial 'flange' frame: attachment point for EEF models -->
-    <link name="${prefix}flange" />
-    <joint name="${prefix}joint_6-flange" type="fixed">
-      <origin xyz="0 0 0" rpy="0 0 0" />
-      <parent link="${prefix}link_6" />
-      <child link="${prefix}flange" />
-    </joint>
-    <!-- ROS-Industrial 'tool0' frame: all-zeros tool frame -->
-<!--    <link name="${prefix}tool0" />-->
-<!--    <joint name="${prefix}link_6-tool0" type="fixed">-->
-<!--      <origin xyz="0 0 0" rpy="${pi} ${-pi/2.0} 0" />-->
-<!--      <parent link="${prefix}flange" />-->
-<!--      <child link="${prefix}tool0" />-->
-<!--    </joint>-->
-  </xacro:macro>
+    <xacro:include filename="$(find fanuc_resources)/urdf/common_materials.xacro"/>
+    <xacro:macro name="fanuc_lrmate200id" params="prefix">
+        <!-- links: main serial chain -->
+        <link name="${prefix}base_link">
+            <visual>
+                <origin xyz="0 0 0" rpy="0 0 0"/>
+                <geometry>
+                    <mesh filename="package://fanuc_lrmate200id_support/meshes/lrmate200id/visual/base_link.stl"/>
+                </geometry>
+                <xacro:material_fanuc_gray28/>
+            </visual>
+            <collision>
+                <origin xyz="0 0 0" rpy="0 0 0"/>
+                <geometry>
+                    <mesh filename="package://fanuc_lrmate200id_support/meshes/lrmate200id/collision/base_link.stl"/>
+                </geometry>
+            </collision>
+        </link>
+        <link name="${prefix}link_1">
+            <visual>
+                <origin xyz="0 0 0" rpy="0 0 0"/>
+                <geometry>
+                    <mesh filename="package://fanuc_lrmate200id_support/meshes/lrmate200id/visual/link_1.stl"/>
+                </geometry>
+                <xacro:material_fanuc_yellow/>
+            </visual>
+            <collision>
+                <origin xyz="0 0 0" rpy="0 0 0"/>
+                <geometry>
+                    <mesh filename="package://fanuc_lrmate200id_support/meshes/lrmate200id/collision/link_1.stl"/>
+                </geometry>
+            </collision>
+        </link>
+        <link name="${prefix}link_2">
+            <visual>
+                <origin xyz="0 0 0" rpy="0 0 0"/>
+                <geometry>
+                    <mesh filename="package://fanuc_lrmate200id_support/meshes/lrmate200id/visual/link_2.stl"/>
+                </geometry>
+                <xacro:material_fanuc_yellow/>
+            </visual>
+            <collision>
+                <origin xyz="0 0 0" rpy="0 0 0"/>
+                <geometry>
+                    <mesh filename="package://fanuc_lrmate200id_support/meshes/lrmate200id/collision/link_2.stl"/>
+                </geometry>
+            </collision>
+        </link>
+        <link name="${prefix}link_3">
+            <visual>
+                <origin xyz="0 0 0" rpy="0 0 0"/>
+                <geometry>
+                    <mesh filename="package://fanuc_lrmate200id_support/meshes/lrmate200id/visual/link_3.stl"/>
+                </geometry>
+                <xacro:material_fanuc_yellow/>
+            </visual>
+            <collision>
+                <origin xyz="0 0 0" rpy="0 0 0"/>
+                <geometry>
+                    <mesh filename="package://fanuc_lrmate200id_support/meshes/lrmate200id/collision/link_3.stl"/>
+                </geometry>
+            </collision>
+        </link>
+        <link name="${prefix}link_4">
+            <visual>
+                <origin xyz="0 0 0" rpy="0 0 0"/>
+                <geometry>
+                    <mesh filename="package://fanuc_lrmate200id_support/meshes/lrmate200id/visual/link_4.stl"/>
+                </geometry>
+                <xacro:material_fanuc_yellow/>
+            </visual>
+            <collision>
+                <origin xyz="0 0 0" rpy="0 0 0"/>
+                <geometry>
+                    <mesh filename="package://fanuc_lrmate200id_support/meshes/lrmate200id/collision/link_4.stl"/>
+                </geometry>
+            </collision>
+        </link>
+        <link name="${prefix}link_5">
+            <visual>
+                <origin xyz="0 0 0" rpy="0 0 0"/>
+                <geometry>
+                    <mesh filename="package://fanuc_lrmate200id_support/meshes/lrmate200id/visual/link_5.stl"/>
+                </geometry>
+                <xacro:material_fanuc_yellow/>
+            </visual>
+            <collision>
+                <origin xyz="0 0 0" rpy="0 0 0"/>
+                <geometry>
+                    <mesh filename="package://fanuc_lrmate200id_support/meshes/lrmate200id/collision/link_5.stl"/>
+                </geometry>
+            </collision>
+        </link>
+        <link name="${prefix}link_6">
+            <visual>
+                <origin xyz="0 0 0" rpy="0 0 0"/>
+                <geometry>
+                    <mesh filename="package://fanuc_lrmate200id_support/meshes/lrmate200id/visual/link_6.stl"/>
+                </geometry>
+                <xacro:material_fanuc_black/>
+            </visual>
+            <collision>
+                <origin xyz="0 0 0" rpy="0 0 0"/>
+                <geometry>
+                    <mesh filename="package://fanuc_lrmate200id_support/meshes/lrmate200id/collision/link_6.stl"/>
+                </geometry>
+            </collision>
+        </link>
+        <!-- joints: main serial chain -->
+        <joint name="${prefix}joint_1" type="revolute">
+            <origin xyz="0 0 0.330" rpy="0 0 0"/>
+            <parent link="${prefix}base_link"/>
+            <child link="${prefix}link_1"/>
+            <axis xyz="0 0 1"/>
+            <limit effort="0" lower="-2.965" upper="2.965" velocity="7.85"/>
+        </joint>
+        <joint name="${prefix}joint_2" type="revolute">
+            <origin xyz="0.050 0 0" rpy="0 0 0"/>
+            <parent link="${prefix}link_1"/>
+            <child link="${prefix}link_2"/>
+            <axis xyz="0 1 0"/>
+            <limit effort="0" lower="-1.745329" upper="2.530727" velocity="6.63"/>
+        </joint>
+        <joint name="${prefix}joint_3" type="revolute">
+            <origin xyz="0 0 0.330" rpy="0 0 0"/>
+            <parent link="${prefix}link_2"/>
+            <child link="${prefix}link_3"/>
+            <axis xyz="0 -1 0"/>
+            <limit effort="0" lower="-2.450966" upper="4.886922" velocity="9.08"/>
+        </joint>
+        <joint name="${prefix}joint_4" type="revolute">
+            <origin xyz="0 0 0.035" rpy="0 0 0"/>
+            <parent link="${prefix}link_3"/>
+            <child link="${prefix}link_4"/>
+            <axis xyz="-1 0 0"/>
+            <limit effort="0" lower="-3.315" upper="3.315" velocity="9.60"/>
+        </joint>
+        <joint name="${prefix}joint_5" type="revolute">
+            <origin xyz="0.335 0 0" rpy="0 0 0"/>
+            <parent link="${prefix}link_4"/>
+            <child link="${prefix}link_5"/>
+            <axis xyz="0 -1 0"/>
+            <limit effort="0" lower="-2.18" upper="2.18" velocity="9.51"/>
+        </joint>
+        <joint name="${prefix}joint_6" type="revolute">
+            <origin xyz="0.080 0 0" rpy="0 0 0"/>
+            <parent link="${prefix}link_5"/>
+            <child link="${prefix}link_6"/>
+            <axis xyz="-1 0 0"/>
+            <limit effort="0" lower="-6.285" upper="6.285" velocity="17.45"/>
+        </joint>
+        <!-- ROS-Industrial 'base' frame: base_link to Fanuc World Coordinates transform -->
+        <link name="${prefix}base"/>
+        <joint name="${prefix}base_link-base" type="fixed">
+            <origin xyz="0 0 0.330" rpy="0 0 0"/>
+            <parent link="${prefix}base_link"/>
+            <child link="${prefix}base"/>
+        </joint>
+        <!-- ROS-Industrial 'flange' frame: attachment point for EEF models -->
+        <link name="${prefix}flange"/>
+        <joint name="${prefix}joint_6-flange" type="fixed">
+            <origin xyz="0 0 0" rpy="0 0 0"/>
+            <parent link="${prefix}link_6"/>
+            <child link="${prefix}flange"/>
+        </joint>
+        <!-- ROS-Industrial 'tool0' frame: all-zeros tool frame -->
+        <link name="${prefix}tool0"/>
+        <joint name="${prefix}link_6-tool0" type="fixed">
+            <origin xyz="0 0 0" rpy="${pi} ${-pi/2.0} 0"/>
+            <parent link="${prefix}flange"/>
+            <child link="${prefix}tool0"/>
+        </joint>
+    </xacro:macro>
 </robot>

File: fanuc_experimental/fanuc_lrmate200id_support/urdf/spray_tool.xacro (robot description, xacro)
@@ -1,30 +1,26 @@
 <?xml version="1.0" encoding="utf-8"?>
 <robot xmlns:xacro="http://ros.org/wiki/xacro">
-  <xacro:macro name="spray_tool" params="prefix connected_to">
-    <!-- Create a fixed joint with a parameterized name. -->
-    <joint name="${prefix}spray_tool_joint" type="fixed">
-<!-- Copied from original data    <parent link="${connected_to}"/> -->
-      <parent link="${prefix}flange"/>
-      <child link="${prefix}spray_tool"/>
-      <origin rpy="${-pi/2} 0 ${pi}" xyz="0 0 0"/>
-    </joint>
-    <link name="${prefix}spray_tool">
-      <visual>
-        <geometry>
-          <mesh filename="file://$(find fanuc_lrmate200id_support)/meshes/lrmate200id/visual/spray_tool.stl" scale="0.001 0.001 0.001"/>
-        </geometry>
-      </visual>
-<!--      <collision>-->
-<!--        <geometry>-->
-<!--          <mesh filename="file://$(find fanuc_lrmate200id_support)/meshes/lrmate200id/visual/spray_tool.stl" scale="0.001 0.001 0.001"/>-->
-<!--        </geometry>-->
-<!--      </collision>-->
-    </link>
-    <joint name="${prefix}tcp_joint" type="fixed">
-      <origin xyz="-0.0758 0 0.2" rpy="0 0 0"/>
-      <parent link="${prefix}spray_tool"/>
-      <child link="${prefix}tcp"/>
-    </joint>
-    <link name="${prefix}tcp"/>
-  </xacro:macro>
+    <xacro:macro name="spray_tool" params="prefix connected_to">
+        <!-- Create a fixed joint with a parameterized name. -->
+        <joint name="${prefix}spray_tool_joint" type="fixed">
+            <!-- Copied from original data    <parent link="${connected_to}"/> -->
+            <parent link="${prefix}tool0"/>
+            <child link="${prefix}spray_tool"/>
+            <origin rpy="0 ${pi/2.0} ${pi/2}" xyz="0 0 0"/>
+        </joint>
+        <link name="${prefix}spray_tool">
+            <visual>
+                <geometry>
+                    <mesh filename="file://$(find fanuc_lrmate200id_support)/meshes/lrmate200id/visual/spray_tool.stl"
+                          scale="0.001 0.001 0.001"/>
+                </geometry>
+            </visual>
+            <collision>
+                <geometry>
+                    <mesh filename="file://$(find fanuc_lrmate200id_support)/meshes/lrmate200id/visual/spray_tool.stl"
+                          scale="0.001 0.001 0.001"/>
+                </geometry>
+            </collision>
+        </link>
+    </xacro:macro>
 </robot>
